File: docs/kicad/gas-detector-mq/gas-detector-mq.kicad_sch (KiCad schematic)
At the start: 8 parts, among them U1 ESP32_DevKit_V1, U2 MH-MQ-Sensor

Commit message: Update schematic revision and adjust designators in KiCad files
Connections:
- net AO_3V3: now also R3.1, R4.2, U1.7 (GPIO32)
- removed net DO_3V3: R3.1, R4.1, U1.7 (GPIO32)
- net GND: no longer names the net of C1.2, C2.2, R2.2, U1.14 (GND), U2.2 (GND)
- net GND: now also R4.1; no longer R4.2, U1.17 (GND), U1.23 (GND)
- no-connect marks 24 -> 28
Other:
- moved on the sheet: C1, C2, R1, R2, R3, R4, U1, U2

Commit message: Add power flag symbol to schematic and adjust wire connections
Connections:
- net AO_3V3: no longer R3.1, R4.2, U1.7 (GPIO32)
- new net DO_3V3: R3.1, R4.2, U1.7 (GPIO32)
Changed lines of the file:
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@@
 	)
 	(junction
-		(at 177.8 160.02)
+		(at 182.88 177.8)
 		(diameter 0)
 		(color 0 0 0 0)
@@
 	(wire
 		(pts
-			(xy 171.45 177.8) (xy 185.42 177.8)
+			(xy 171.45 177.8) (xy 182.88 177.8)
 		)
 		(stroke
@@
 	(wire
 		(pts
-			(xy 241.3 138.43) (xy 144.78 138.43)
+			(xy 229.87 138.43) (xy 144.78 138.43)
 		)
 		(stroke
@@
 	(wire
 		(pts
-			(xy 177.8 154.94) (xy 177.8 160.02)
+			(xy 129.54 191.77) (xy 137.16 191.77)
 		)
 		(stroke
@@
 	(wire
 		(pts
-			(xy 129.54 191.77) (xy 137.16 191.77)
+			(xy 182.88 177.8) (xy 185.42 177.8)
+		)
+		(stroke
+			(width 0)
+			(type default)
+			(color 0 0 0 1)
+		)
+	)
+	(wire
+		(pts
+			(xy 134.62 154.94) (xy 144.78 154.94)
+		)
+		(stroke
+			(width 0)
+			(type default)
+			(color 255 0 0 1)
+		)
+	)
+	(wire
+		(pts
+			(xy 106.68 154.94) (xy 134.62 154.94)
+		)
+		(stroke
+			(width 0)
+			(type default)
+			(color 255 0 0 1)
+		)
+	)
+	(wire
+		(pts
+			(xy 137.16 191.77) (xy 137.16 217.17)
 		)
 		(stroke
@@
 	(wire
 		(pts
-			(xy 134.62 154.94) (xy 144.78 154.94)
+			(xy 153.67 160.02) (xy 185.42 160.02)
+		)
+		(stroke
+			(width 0)
+			(type default)
+			(color 132 132 0 1)
+		)
+	)
+	(wire
+		(pts
+			(xy 91.44 162.56) (xy 91.44 168.91)
+		)
+		(stroke
+			(width 0)
+			(type default)
+			(color 0 0 0 1)
+		)
+	)
+	(wire
+		(pts
+			(xy 129.54 189.23) (xy 146.05 189.23)
+		)
+		(stroke
+			(width 0)
+			(type default)
+			(color 132 132 0 1)
+		)
+	)
+	(wire
+		(pts
+			(xy 137.16 217.17) (xy 161.29 217.17)
+		)
+		(stroke
+			(width 0)
+			(type default)
+			(color 132 0 132 1)
+		)
+	)
+	(wire
+		(pts
+			(xy 134.62 184.15) (xy 129.54 184.15)
 		)
 		(stroke
@@
 	(wire
 		(pts
-			(xy 106.68 154.94) (xy 134.62 154.94)
+			(xy 162.56 177.8) (xy 171.45 177.8)
+		)
+		(stroke
+			(width 0)
+			(type default)
+			(color 0 0 0 1)
+		)
+	)
+	(wire
+		(pts
+			(xy 226.06 144.78) (xy 229.87 144.78)
 		)
 		(stroke
@@
 	(wire
 		(pts
-			(xy 137.16 191.77) (xy 137.16 217.17)
+			(xy 161.29 189.23) (xy 171.45 189.23)
+		)
+		(stroke
+			(width 0)
+			(type default)
+			(color 0 0 0 1)
+		)
+	)
+	(wire
+		(pts
+			(xy 229.87 144.78) (xy 229.87 138.43)
+		)
+		(stroke
+			(width 0)
+			(type default)
+			(color 255 0 0 1)
+		)
+	)
+	(wire
+		(pts
+			(xy 171.45 217.17) (xy 177.8 217.17)
 		)
 		(stroke
@@
 	(wire
 		(pts
-			(xy 153.67 160.02) (xy 177.8 160.02)
+			(xy 177.8 154.94) (xy 177.8 217.17)
+		)
+		(stroke
+			(width 0)
+			(type default)
+			(color 132 0 132 1)
+		)
+	)
+	(wire
+		(pts
+			(xy 91.44 168.91) (xy 106.68 168.91)
+		)
+		(stroke
+			(width 0)
+			(type default)
+			(color 0 0 0 1)
+		)
+	)
+	(wire
+		(pts
+			(xy 153.67 160.02) (xy 153.67 189.23)
 		)
 		(stroke
@@
 	(wire
 		(pts
-			(xy 91.44 162.56) (xy 91.44 168.91)
-		)
-		(stroke
-			(width 0)
-			(type default)
-			(color 0 0 0 1)
-		)
-	)
-	(wire
-		(pts
-			(xy 129.54 189.23) (xy 146.05 189.23)
-		)
-		(stroke
-			(width 0)
-			(type default)
-			(color 132 132 0 1)
-		)
-	)
-	(wire
-		(pts
-			(xy 137.16 217.17) (xy 161.29 217.17)
+			(xy 185.42 154.94) (xy 177.8 154.94)
 		)
 		(stroke
@@
 		)
 	)
-	(wire
-		(pts
-			(xy 134.62 184.15) (xy 129.54 184.15)
-		)
-		(stroke
-			(width 0)
-			(type default)
-			(color 255 0 0 1)
-		)
-	)
-	(wire
-		(pts
-			(xy 162.56 177.8) (xy 171.45 177.8)
-		)
-		(stroke
-			(width 0)
-			(type default)
-			(color 0 0 0 1)
-		)
-	)
-	(wire
-		(pts
-			(xy 226.06 144.78) (xy 241.3 144.78)
-		)
-		(stroke
-			(width 0)
-			(type default)
-			(color 255 0 0 1)
-		)
-	)
-	(wire
-		(pts
-			(xy 161.29 189.23) (xy 171.45 189.23)
-		)
-		(stroke
-			(width 0)
-			(type default)
-			(color 0 0 0 1)
-		)
-	)
-	(wire
-		(pts
-			(xy 241.3 144.78) (xy 241.3 138.43)
-		)
-		(stroke
-			(width 0)
-			(type default)
-			(color 255 0 0 1)
-		)
-	)
-	(wire
-		(pts
-			(xy 171.45 217.17) (xy 177.8 217.17)
-		)
-		(stroke
-			(width 0)
-			(type default)
-			(color 132 0 132 1)
-		)
-	)
-	(wire
-		(pts
-			(xy 177.8 160.02) (xy 177.8 217.17)
-		)
-		(stroke
-			(width 0)
-			(type default)
-			(color 132 0 132 1)
-		)
-	)
-	(wire
-		(pts
-			(xy 91.44 168.91) (xy 106.68 168.91)
-		)
-		(stroke
-			(width 0)
-			(type default)
-			(color 0 0 0 1)
-		)
-	)
-	(wire
-		(pts
-			(xy 153.67 160.02) (xy 153.67 189.23)
-		)
-		(stroke
-			(width 0)
-			(type default)
-			(color 132 132 0 1)
-		)
-	)
-	(wire
-		(pts
-			(xy 185.42 154.94) (xy 177.8 154.94)
-		)
-		(stroke
-			(width 0)
-			(type default)
-		)
-	)
-	(wire
-		(pts
-			(xy 177.8 160.02) (xy 185.42 160.02)
-		)
-		(stroke
-			(width 0)
-			(type default)
-			(color 132 132 0 1)
-		)
-	)
 	(label "+5V"
-		(at 241.3 144.78 0)
+		(at 229.87 144.78 0)
 		(effects
 			(font
@@
 		)
 	)
-	(label "DO_3V3"
-		(at 177.8 160.02 0)
-		(effects
-			(font
-				(size 1.27 1.27)
-			)
-			(justify left bottom)
-		)
-	)
 	(label "+5V"
 		(at 144.78 154.94 0)
@@
 			(font
 				(size 1.27 1.27)
-			)
-			(justify left bottom)
-		)
-	)
-	(label "AO_3V3"
-		(at 177.8 154.94 0)
-		(effects
-			(font
-				(size 1.27 1.27)
-				(color 132 0 132 1)
 			)
 			(justify left bottom)
@@
 					(unit 1)
 				)
+			)
+		)
+	)
+	(symbol
+		(lib_id "power:PWR_FLAG")
+		(at 182.88 177.8 0)
+		(unit 1)
+		(body_style 1)
+		(exclude_from_sim no)
+		(in_bom yes)
+		(on_board yes)
+		(in_pos_files yes)
+		(dnp no)
+		(fields_autoplaced yes)
+		(property "Reference" "#FLG01"
+			(at 182.88 175.895 0)
+			(hide yes)
+			(show_name no)
+			(do_not_autoplace no)
+			(effects
+				(font
+					(size 1.27 1.27)
+				)
+			)
+		)
+		(property "Value" "PWR_FLAG"
+			(at 182.88 172.72 0)
+			(show_name no)
+			(do_not_autoplace no)
+			(effects
+				(font
+					(size 1.27 1.27)
+				)
+			)
+		)
+		(property "Footprint" ""
+			(at 182.88 177.8 0)
+			(hide yes)
+			(show_name no)
+			(do_not_autoplace no)
+			(effects
+				(font
+					(size 1.27 1.27)
+				)
+			)
+		)
+		(property "Datasheet" ""
+			(at 182.88 177.8 0)
+			(hide yes)
+			(show_name no)
+			(do_not_autoplace no)
+			(effects
+				(font
+					(size 1.27 1.27)
+				)
+			)
+		)
+		(property "Description" "Special symbol for telling ERC where power comes from"
+			(at 182.88 177.8 0)
+			(hide yes)
+			(show_name no)
+			(do_not_autoplace no)
+			(effects
+				(font
+					(size 1.27 1.27)
+				)
+			)
+		)
+		(pin "1"
+		)
+		(instances
+			(project "gas-detector-mq"
+				(path "/2f6c1a84-7b3e-4d19-9c55-0a8e4b71d2c6"
+					(reference "#FLG01")
+					(unit 1)
+				)
