File: docs/kicad/gas-detector-mq/gas-detector-mq.kicad_sch (KiCad schematic)
At the start: 8 parts, among them U1 ESP32_DevKit_V1, U2 MH-MQ-Sensor

Commit message: Zostaw na prototypie bulk 10 µF / 50 V.
Ten kondensator jest już pod ręką. 47 µF / 50 V zostaje zakupem na później.

Co-authored-by: michal.kalkowski <michal.kalkowski@sumup.com>
Parts:
- C2: value 47uF -> 10uF
Other:
- note added: "Prototyp na płytce uniwersalnej — bez PCB. USB zasila ESP32. Moduł MQ z pinu 5V/VIN (grzałka ~150 mA, potrzebuje 5 V, nie 3V3). AO 5 V → R1 10k → węzeł → GPIO34/D34 (ADC1_CH6); węzeł → R2 20k → GND. DO 5 V → R3 10k → węzeł → GPIO35/D35; węzeł → R4 20k → GND. Na pinie jest 3,33 V. C1 100 nF i C2 10 µF/50 V przy VCC modułu. Krzyżyki: tych pinów nie lutować. Złącze MQ: VCC, GND, DO, AO — sprawdź nad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"
- note removed: "Prototyp na płytce uniwersalnej — bez PCB. USB zasila ESP32. Moduł MQ z pinu 5V/VIN (grzałka ~150 mA, potrzebuje 5 V, nie 3V3). AO 5 V → R1 10k → węzeł → GPIO34/D34 (ADC1_CH6); węzeł → R2 20k → GND. DO 5 V → R3 10k → węzeł → GPIO35/D35; węzeł → R4 20k → GND. Na pinie jest 3,33 V. C1 100 nF i C2 47 µF/50 V przy VCC modułu. Krzyżyki: tych pinów nie lutować. Złącze MQ: VCC, GND, DO, AO — sprawdź nad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"
Changed lines of the file:
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@@
 		(comment 3 "Założenie: DOIT DevKit V1 30 pin, USB na dole; złącze MQ VCC GND DO AO.")
 	)
-	(text "Prototyp na płytce uniwersalnej — bez PCB.\nUSB zasila ESP32. Moduł MQ z pinu 5V/VIN (grzałka ~150 mA, potrzebuje 5 V, nie 3V3).\nAO 5 V → R1 10k → węzeł → GPIO34/D34 (ADC1_CH6); węzeł → R2 20k → GND.\nDO 5 V → R3 10k → węzeł → GPIO35/D35; węzeł → R4 20k → GND. Na pinie jest 3,33 V.\nC1 100 nF i C2 47 µF/50 V przy VCC modułu. Krzyżyki: tych pinów nie lutować.\nZłącze MQ: VCC, GND, DO, AO — sprawdź nadruk. DevKit 30 pin, USB na dole;\nlewy rząd od 3V3, prawy od VIN. Przed lutowaniem porównaj z nadrukiem płytki."
+	(text "Prototyp na płytce uniwersalnej — bez PCB.\nUSB zasila ESP32. Moduł MQ z pinu 5V/VIN (grzałka ~150 mA, potrzebuje 5 V, nie 3V3).\nAO 5 V → R1 10k → węzeł → GPIO34/D34 (ADC1_CH6); węzeł → R2 20k → GND.\nDO 5 V → R3 10k → węzeł → GPIO35/D35; węzeł → R4 20k → GND. Na pinie jest 3,33 V.\nC1 100 nF i C2 10 µF/50 V przy VCC modułu. Krzyżyki: tych pinów nie lutować.\nZłącze MQ: VCC, GND, DO, AO — sprawdź nadruk. DevKit 30 pin, USB na dole;\nlewy rząd od 3V3, prawy od VIN. Przed lutowaniem porównaj z nadrukiem płytki."
 		(exclude_from_sim no)
 		(at 301.752 236.474 0)
@@
 			)
 		)
-		(property "Value" "47uF"
+		(property "Value" "10uF"
 			(at 111.76 161.29 0)
 			(show_name no)
